File: Código_Agos_BLUEPAD32/Placa_Futboleros/Placa_Futboleros_Nueva/Placa V3/Placa_Futboleros_Nueva.kicad_pcb (KiCad board)
At the start: 2 copper layers, 52 x 100.8 mm, 17 parts, among them J1 BAT, J2 Motor_Izq_Adelante, J3 Motor_Izq_Atras, J4 Motor_Der_Adelante, J5 Motor_Der_Atras, U1 AMS1117, U2 esp32_36_pins-custom_library, U3 DRV8833, U4 DRV8833

Commit message: Nueva versión de Código
El mismo incluye manejo con botones y comentarios que describen los cambios de pines
entre futboleros, de forma que se actualice el código cada vez que se cambie de
robot
Parts:
- moved J1 1.73 mm to (176.1, 126.9)
Routing:
- net GND: track 216.3 -> 213.9 mm
- net VCC: track 99.0 -> 98.3 mm, vias 3 -> 2
Other:
- board size 52 x 100.8 mm -> 52 x 100 mm
Changed lines of the file:
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@@
 			(at 0 0)
 			(size 3 3)
-			(drill 3)
+			(drill 0.1)
 			(layers "*.Cu" "*.Mask")
 		)
@@
 		(tags "C Radial series Radial pin pitch 5.00mm diameter 10mm height 12.5mm Non-Polar Electrolytic Capacitor")
 		(property "Reference" "C1"
-			(at 2.5 0 90)
+			(at 9.064 0 180)
 			(layer "F.SilkS")
 			(effects
@@
 		)
 		(fp_text user "${REFERENCE}"
-			(at 2.5 0 90)
+			(at 7.5 0 180)
 			(layer "F.Fab")
 			(effects
@@
 			(at 0 0)
 			(size 3 3)
-			(drill 3)
+			(drill 0.1)
 			(layers "*.Cu" "*.Mask")
 		)
@@
 		(at 180.14923 95.950694 -90)
 		(property "Reference" "U3"
-			(at 0 -0.5 270)
+			(at -10.668 -10.16 0)
 			(unlocked yes)
 			(layer "F.SilkS")
@@
 			(at 0 0)
 			(size 3 3)
-			(drill 3)
+			(drill 0.1)
 			(layers "*.Cu" "*.Mask")
 		)
@@
 		(tags "Through hole socket strip THT 1x18 2.54mm single row")
 		(property "Reference" "U2"
-			(at 0 -2.77 0)
+			(at 0.508 -7.112 180)
 			(layer "F.SilkS")
 			(effects
@@
 		(tags "Diode DO-41_SOD81 series Axial Horizontal pin pitch 10.16mm  length 5.2mm diameter 2.7mm")
 		(property "Reference" "D1"
-			(at 5.08 -2.47 90)
+			(at 0 3.556 180)
 			(layer "F.SilkS")
 			(effects
@@
 		)
 		(fp_text user "K"
-			(at 0 -2.1 90)
+			(at 0 -3.048 180)
 			(layer "F.SilkS")
 			(effects
@@
 	(footprint "Connector_JST:JST_EH_B2B-EH-A_1x02_P2.50mm_Vertical"
 		(layer "F.Cu")
-		(at 176.08523 128.670694 180)
+		(at 176.08523 126.938694 180)
 		(descr "JST EH series connector, B2B-EH-A (http://www.jst-mfg.com/product/pdf/eng/eEH.pdf)")
 		(tags "connector JST EH vertical")
 		(property "Reference" "J1"
-			(at 1.25 -2.8 0)
+			(at -4.064 2.24 0)
 			(layer "F.SilkS")
 			(effects
@@
 		(property "Value" "BAT"
 			(at 1.25 3.4 0)
-			(layer "F.Fab")
+			(layer "F.SilkS")
 			(effects
 				(font
@@
 		(tags "Resistor Axial_DIN0207 series Axial Horizontal pin pitch 10.16mm 0.25W = 1/4W length 6.3mm diameter 2.5mm")
 		(property "Reference" "R1"
-			(at 5.08 -2.37 90)
+			(at 12.192 0 180)
 			(layer "F.SilkS")
 			(effects
@@
 		(at 200.46923 66.994694 90)
 		(property "Reference" "U4"
-			(at 0 -0.5 90)
+			(at 10.668 -9.652 0)
 			(unlocked yes)
 			(layer "F.SilkS")
@@
 			(at 0 0)
 			(size 3 3)
-			(drill 3)
+			(drill 0.1)
 			(layers "*.Cu" "*.Mask")
 		)
@@
 	)
 	(gr_rect
-		(start 149.48523 31.434694)
-		(end 201.48523 132.234694)
+		(start 149.57723 29.986694)
+		(end 201.57723 129.986694)
 		(stroke
 			(width 0.07)
@@
 	)
 	(segment
+		(start 181.16523 112.714694)
+		(end 181.16523 94.934694)
+		(width 1.2)
+		(layer "F.Cu")
+		(net "GND")
+	)
+	(segment
 		(start 183.19723 78.170694)
 		(end 181.16523 80.202694)
@@
 	)
 	(segment
-		(start 181.16523 94.934694)
-		(end 181.16523 112.714694)
-		(width 1.2)
-		(layer "F.Cu")
-		(net "GND")
-	)
-	(segment
 		(start 181.497805 94.251269)
 		(end 181.67323 94.251269)
@@
 	)
 	(segment
-		(start 181.16523 112.714694)
-		(end 173.54523 120.334694)
+		(start 181.16523 93.918694)
+		(end 181.497805 94.251269)
 		(width 1.2)
 		(layer "F.Cu")
@@
 	(segment
 		(start 173.54523 120.334694)
-		(end 173.54523 123.382694)
-		(width 1.2)
-		(layer "F.Cu")
-		(net "GND")
-	)
-	(segment
-		(start 181.16523 93.918694)
-		(end 181.497805 94.251269)
+		(end 181.16523 112.714694)
 		(width 1.2)
 		(layer "F.Cu")
@@
 	)
 	(via
-		(at 173.54523 123.382694)
+		(at 173.54523 120.334694)
 		(size 2.6)
 		(drill 0.8)
@@
 	)
 	(segment
-		(start 173.54523 123.382694)
-		(end 173.54523 128.630694)
+		(start 156.78123 120.334694)
+		(end 163.38523 126.938694)
 		(width 1.2)
 		(layer "B.Cu")
@@
 	)
 	(segment
-		(start 165.11723 128.670694)
-		(end 173.58523 128.670694)
+		(start 173.54523 120.334694)
+		(end 173.54523 126.898694)
 		(width 1.2)
 		(layer "B.Cu")
@@
 	)
 	(segment
-		(start 173.54523 128.630694)
-		(end 173.58523 128.670694)
-		(width 1.2)
-		(layer "B.Cu")
-		(net "GND")
-	)
-	(segment
-		(start 156.78123 120.334694)
-		(end 165.11723 128.670694)
+		(start 173.54523 126.898694)
+		(end 173.58523 126.938694)
 		(width 1.2)
 		(layer "B.Cu")
@@
 	)
 	(segment
+		(start 163.38523 126.938694)
+		(end 173.58523 126.938694)
+		(width 1.2)
+		(layer "B.Cu")
+		(net "GND")
+	)
+	(segment
 		(start 153.22523 108.650694)
 		(end 155.76523 106.110694)
@@
 	)
 	(via
-		(at 197.59123 121.520694)
-		(size 2.6)
-		(drill 0.8)
-		(layers "F.Cu" "B.Cu")
-		(net "VCC")
-	)
-	(via
 		(at 192.84923 78.170694)
 		(size 2.6)
@@
 	)
 	(segment
-		(start 190.60923 128.670694)
-		(end 193.86523 125.414694)
+		(start 191.83323 77.154694)
+		(end 191.83323 74.868694)
 		(width 1.2)
 		(layer "B.Cu")
@@
 	)
 	(segment
-		(start 191.83323 77.154694)
-		(end 191.83323 74.868694)
+		(start 192.34123 126.938694)
+		(end 193.86523 125.414694)
 		(width 1.2)
 		(layer "B.Cu")
@@
 	)
 	(segment
-		(start 176.08523 128.670694)
-		(end 190.60923 128.670694)
+		(start 176.08523 126.938694)
+		(end 192.34123 126.938694)
 		(width 1.2)
 		(layer "B.Cu")
