File: Placa_Futboleros/Placa_Futboleros/Placa V4/Corrección/Placa V4_Corrección.kicad_sch (KiCad schematic)
At the start: 31 parts, among them J1 LiPo, J2 MI_Ad, J3 MI_At, J4 MD_Ad, J5 MD_At, J6 Pilas, U1 ESP32_30p, U2 DRV8833, U3 DRV8833, U5 INA219AxD

Commit message: Pusheo de archivos varios del SementalItaliano
1. Diseños de solid edge del robot:
  - Se utiliza ahora únicamente dos motores más potentes.
  - Eso requiere un sistema de engranajes, donde los ejes de las ruedas de atrás
  son del motor, hay engranajes bobos en medio y luego las ruedas delanteras.
  - Se agrega la llave en la tapa para ON-OFF del robot.
  - La LiPo es más grande.

2. Cambio de LiPo a una de 14,8V 2200mAh con 45C.
3. Se rehace por ese motivo la placa, con drivers BTS7960, así que se redistribuye cosas
en el robot, y se agrega para montar y desmontar el módulo de la placa.
4. Las placas tiene 1,7mm de ancho de pista grande y 0,8 creo de pistas chicas; hay solo dos puentes,
uno chiquito y otro corto pero de cable grueso, se adaptó el orificio para que pase bien el cable.
Connections:
- net IN_M1A: now also U1.14 (D22); no longer U1.23 (D25)
- net IN_M1B: now also U1.11 (D21); no longer U1.24 (D26)
- net SLEEP_M1: now also U1.15 (D23); no longer U1.6 (RX2)
- net SLEEP_M2: now also U1.6 (RX2); no longer U1.15 (D23)
